Commit message: .obj to .stl

File: res/model.urdf (robot description, URDF)
Before this commit: robot iCubHAND, 26 links, 25 joints
Links:
- link l_hand: geometry visual mesh filename=package://iCub/meshes/full_LeftTopCoverMarker.stl scale=0.001 0.001 0.001
- link l_hand_index_0: geometry visual mesh filename=package://iCub/meshes/full_LeftIndex0.stl scale=0.001 0.001 0.001
- link l_hand_index_1: geometry visual mesh filename=package://iCub/meshes/full_LeftIndex1.stl scale=0.001 0.001 0.001
- link l_hand_index_2: geometry visual mesh filename=package://iCub/meshes/full_LeftIndex2.stl scale=0.001 0.001 0.001
- link l_hand_index_3: geometry visual mesh filename=package://iCub/meshes/full_LeftIndex3.stl scale=0.001 0.001 0.001
- link l_hand_little_0: geometry visual mesh filename=package://iCub/meshes/full_LeftLittle0.stl scale=0.001 0.001 0.001
- link l_hand_little_1: geometry visual mesh filename=package://iCub/meshes/full_LeftLittle1.stl scale=0.001 0.001 0.001
- link l_hand_little_2: geometry visual mesh filename=package://iCub/meshes/full_LeftLittle2.stl scale=0.001 0.001 0.001
- link l_hand_little_3: geometry visual mesh filename=package://iCub/meshes/full_LeftLittle3.stl scale=0.001 0.001 0.001
- link l_hand_middle_0: geometry visual mesh filename=package://iCub/meshes/full_LeftMiddle0.stl scale=0.001 0.001 0.001
- link l_hand_middle_1: geometry visual mesh filename=package://iCub/meshes/full_LeftMiddle1.stl scale=0.001 0.001 0.001
- link l_hand_middle_2: geometry visual mesh filename=package://iCub/meshes/full_LeftMiddle2.stl scale=0.001 0.001 0.001
- link l_hand_middle_3: geometry visual mesh filename=package://iCub/meshes/full_LeftMiddle3.stl scale=0.001 0.001 0.001
- link l_hand_ring_0: geometry visual mesh filename=package://iCub/meshes/full_LeftRing0.stl scale=0.001 0.001 0.001
- link l_hand_ring_1: geometry visual mesh filename=package://iCub/meshes/full_LeftRing1.stl scale=0.001 0.001 0.001
- link l_hand_ring_2: geometry visual mesh filename=package://iCub/meshes/full_LeftRing2.stl scale=0.001 0.001 0.001
- link l_hand_ring_3: geometry visual mesh filename=package://iCub/meshes/full_LeftRing3.stl scale=0.001 0.001 0.001
- link l_hand_thumb_0: geometry visual mesh filename=package://iCub/meshes/full_LeftThumb0.stl scale=0.001 0.001 0.001
- link l_hand_thumb_1: geometry visual mesh filename=package://iCub/meshes/full_LeftThumb1.stl scale=0.001 0.001 0.001
- link l_hand_thumb_2: geometry visual mesh filename=package://iCub/meshes/full_LeftThumb2.stl scale=0.001 0.001 0.001
- link l_hand_thumb_3: geometry visual mesh filename=package://iCub/meshes/full_LeftThumb3.stl scale=0.001 0.001 0.001
